Commit message: mesh update

File: ur_description/urdf/ur3.urdf.xacro (robot description, xacro)
@@ -386,37 +386,4 @@
     </joint>
     <xacro:intel_realsense_mount prefix="camera" topic="camera_image" parent_link="camera_link"/>
-  <!-- only for us -->
-    <link name="grasping_frame">
-      <inertial>
-        <origin xyz="0.2 0.2 0.025" rpy="0 0 0"/>
-        <mass value="0.0001"/>
-        <inertia  ixx="1.0" ixy="0.0"  ixz="0.0"  iyy="100.0"  iyz="0.0"  izz="1.0" />
-      </inertial>
-      <collision>
-        <origin xyz="0 0 0" rpy="0 0 0"/>
-        <geometry>
-          <box size="0.05 0.05 0.05"/>
-        </geometry>
-      </collision>
-      <visual>
-        <origin xyz="0.2 0.2 0.025" rpy="0 0 0"/>
-        <geometry>
-          <mesh filename="file://$(find ur_description)/meshes/aruco_cube_5cm.dae"/>
-        </geometry>
-      </visual>
-    </link>
-    <gazebo reference='grasping_frame'>
-      <kp>100000.0</kp>
-      <kd>100000.0</kd>
-      <mu1>0.1</mu1>
-      <mu2>0.1</mu2>
-      <fdir1>1 0 0</fdir1>
-    </gazebo>
-    <joint name="grasping_frame_joint" type="fixed">
-      <parent link="world"/>
-      <child link="grasping_frame"/>
-      <origin xyz="0.2 0.2 0.025" rpy="0 0 0"/>
-    </joint>
-    <!-- only for us -->
   </xacro:macro>
 </robot>
