Commit message: gripper

File: ur_description/urdf/intel_realsense.urdf.xacro (robot description, xacro)
@@ -1,10 +1,10 @@
 <?xml version="1.0"?>
 <robot xmlns:xacro="http://ros.org/wiki/xacro">
-  <xacro:macro name="intel_realsense_mount" params="prefix topic parent_link">
+  <xacro:macro name="camera_mount" params="prefix topic parent_link">
                <!--h_fov:=1.5184351666666667 v_fov:=1.0122901111111111/-->
     <xacro:macro name="intel_realsense" params="
-               frame:=realsense          topic:=realsense
+               frame:=camera             topic:=camera
                h_fov:=1.2112585009       v_fov:=0.7417649321
-               min_range:=0.105          max_range:=8.0
+               min_range:=0.105          max_range:=0.105
                width:=640                height:=480
                update_rate:=30
@@ -25,5 +25,5 @@
       <gazebo reference="${frame}">
         <turnGravityOff>true</turnGravityOff>
-        <sensor type="depth" name="${prefix}_realsense_depth">
+        <sensor type="depth" name="${prefix}_camera_depth">
           <update_rate>${update_rate}</update_rate>
           <camera>
@@ -70,5 +70,5 @@
       </gazebo>
     </xacro:macro>
-    <link name="${prefix}_realsense_lens">
+    <link name="${prefix}_camera_lens">
       <visual>
         <!--
@@ -80,15 +80,15 @@
       </visual>
     </link>
-    <joint type="fixed" name="${prefix}_realsense_lens_joint">
+    <joint type="fixed" name="${prefix}_camera_lens_joint">
       <origin xyz="0 0 0" rpy="0 0 0" />
       <parent link="${parent_link}" />
-      <child link="${prefix}_realsense_lens" />
+      <child link="${prefix}_camera_lens" />
     </joint>
-    <joint type="fixed" name="${prefix}_realsense_joint">
-      <origin xyz="0.025 0 0" rpy="0 0 0" />
-      <parent link="${prefix}_realsense_lens" />
-      <child link="${prefix}_realsense" />
+    <joint type="fixed" name="${prefix}_camera_joint">
+      <origin xyz="0.0 0 0" rpy="-1.5707 0 0" />
+      <parent link="${prefix}_camera_lens" />
+      <child link="${prefix}_camera" />
     </joint>
-    <xacro:intel_realsense frame="${prefix}_realsense" topic="${topic}"/>
+    <xacro:intel_realsense frame="${prefix}_camera" topic="${topic}"/>
   </xacro:macro>
 </robot>

File: ur_description/urdf/ur3.urdf.xacro (robot description, xacro)
@@ -65,4 +65,28 @@
       <color rgba="1 1 1 1"/>
     </material>
+    <material name="Blue">
+      <color rgba="0 0 0.8 1"/>
+    </material>
+    <material name="Red">
+      <color rgba="0.8 0 0 1"/>
+    </material>
+    <material name="Green">
+      <color rgba="0 0.8 0 1"/>
+    </material>
+    <material name="Yellow">
+      <color rgba="0.4 0.4 0 1"/>
+    </material>
+    <material name="Orange">
+      <color rgba="0.8 0.5 0 1"/>
+    </material>
+    <material name="Purple">
+      <color rgba="0.8 0 0.8 1"/>
+    </material>
+    <material name="Grey">
+      <color rgba="0.4 0.4 0.4 1"/>
+    </material>
+    <material name="LightGrey">
+      <color rgba="0.7 0.7 0.7 1"/>
+    </material>
     <link name="${prefix}base_link" >
       <visual>
@@ -83,9 +107,295 @@
       </xacro:cylinder_inertial>
     </link>
+    <joint name="${prefix}shoulder_pan_joint" type="revolute">
+      <parent link="${prefix}base_link" />
+      <child link = "${prefix}shoulder_link" />
+      <origin xyz="0.0 0.0 ${shoulder_height}" rpy="0.0 0.0 0.0" />
+      <axis xyz="0 0 1" />
+      <xacro:unless value="${joint_limited}">
+        <limit lower="${-2.0 * pi}" upper="${2.0 * pi}" effort="330.0" velocity="2.16"/>
+        <xacro:if value="${safety_limits}">
+          <safety_controller soft_lower_limit="${-2.0 * pi + safety_pos_margin}" soft_upper_limit="${2.0 * pi - safety_pos_margin}" k_position="${safety_k_position}" k_velocity="0.0"/>
+        </xacro:if>
+      </xacro:unless>
+      <xacro:if value="${joint_limited}">
+        <limit lower="${shoulder_pan_lower_limit}" upper="${shoulder_pan_upper_limit}" effort="330.0" velocity="2.16"/>
+        <xacro:if value="${safety_limits}">
+          <safety_controller soft_lower_limit="${shoulder_pan_lower_limit + safety_pos_margin}" soft_upper_limit="${shoulder_pan_upper_limit - safety_pos_margin}" k_position="${safety_k_position}" k_velocity="0.0"/>
+        </xacro:if>
+      </xacro:if>
+      <dynamics damping="0.0" friction="0.0"/>
+    </joint>
+    <link name="${prefix}shoulder_link">
+      <visual>
+        <geometry>
+          <mesh filename="package://ur_description/meshes/ur3/visual/shoulder.dae"/>
+        </geometry>
+        <material name="LightGrey">
+          <color rgba="0.7 0.7 0.7 1.0"/>
+        </material>
+      </visual>
+      <collision>
+        <geometry>
+          <mesh filename="package://ur_description/meshes/ur3/collision/shoulder.stl"/>
+        </geometry>
+      </collision>
+      <xacro:cylinder_inertial radius="0.075" length="0.178" mass="${shoulder_mass}">
+        <origin xyz="0.0 0.0 0.0" rpy="0 0 0" />
+      </xacro:cylinder_inertial>
+    </link>
+    <joint name="${prefix}shoulder_lift_joint" type="revolute">
+      <parent link="${prefix}shoulder_link" />
+      <child link = "${prefix}upper_arm_link" />
+      <origin xyz="0.0 ${shoulder_offset} 0.0" rpy="0.0 ${pi / 2.0} 0.0" />
+      <axis xyz="0 1 0" />
+      <xacro:unless value="${joint_limited}">
+        <limit lower="${-2.0 * pi}" upper="${2.0 * pi}" effort="330.0" velocity="2.16"/>
+        <xacro:if value="${safety_limits}">
+          <safety_controller soft_lower_limit="${-2.0 * pi + safety_pos_margin}" soft_upper_limit="${2.0 * pi - safety_pos_margin}" k_position="${safety_k_position}" k_velocity="0.0"/>
+        </xacro:if>
+      </xacro:unless>
+      <xacro:if value="${joint_limited}">
+        <limit lower="${shoulder_lift_lower_limit}" upper="${shoulder_lift_upper_limit}" effort="330.0" velocity="2.16"/>
+        <xacro:if value="${safety_limits}">
+          <safety_controller soft_lower_limit="${shoulder_lift_lower_limit + safety_pos_margin}" soft_upper_limit="${shoulder_lift_upper_limit - safety_pos_margin}" k_position="${safety_k_position}" k_velocity="0.0"/>
+        </xacro:if>
+      </xacro:if>
+      <dynamics damping="0.0" friction="0.0"/>
+    </joint>
+    <link name="${prefix}upper_arm_link">
+      <visual>
+        <geometry>
+          <mesh filename="package://ur_description/meshes/ur3/visual/upperarm.dae"/>
+        </geometry>
+        <material name="LightGrey">
+          <color rgba="0.7 0.7 0.7 1.0"/>
+        </material>
+      </visual>
+      <collision>
+        <geometry>
+          <mesh filename="package://ur_description/meshes/ur3/collision/upperarm.stl"/>
+        </geometry>
+      </collision>
+      <xacro:cylinder_inertial radius="0.075" length="${-a2}" mass="${upper_arm_mass}">
+        <origin xyz="0.0 0.0 ${-a2/2.0}" rpy="0 0 0" />
+      </xacro:cylinder_inertial>
+    </link>
+    <joint name="${prefix}elbow_joint" type="revolute">
+      <parent link="${prefix}upper_arm_link" />
+      <child link = "${prefix}forearm_link" />
+      <origin xyz="0.0 ${elbow_offset} ${upper_arm_length}" rpy="0.0 0.0 0.0" />
+      <axis xyz="0 1 0" />
+      <xacro:unless value="${joint_limited}">
+        <limit lower="${-pi}" upper="${pi}" effort="150.0" velocity="3.15"/>
+        <xacro:if value="${safety_limits}">
+          <safety_controller soft_lower_limit="${-2.0 * pi + safety_pos_margin}" soft_upper_limit="${2.0 * pi - safety_pos_margin}" k_position="${safety_k_position}" k_velocity="0.0"/>
+        </xacro:if>
+      </xacro:unless>
+      <xacro:if value="${joint_limited}">
+        <limit lower="${elbow_joint_lower_limit}" upper="${elbow_joint_upper_limit}" effort="150.0" velocity="3.15"/>
+        <xacro:if value="${safety_limits}">
+          <safety_controller soft_lower_limit="${elbow_joint_lower_limit + safety_pos_margin}" soft_upper_limit="${elbow_joint_upper_limit - safety_pos_margin}" k_position="${safety_k_position}" k_velocity="0.0"/>
+        </xacro:if>
+      </xacro:if>
+      <dynamics damping="0.0" friction="0.0"/>
+    </joint>
+    <link name="${prefix}forearm_link">
+      <visual>
+         <geometry>
+          <mesh filename="package://ur_description/meshes/ur3/visual/forearm.dae"/>
+        </geometry>
+        <material name="LightGrey">
+          <color rgba="0.7 0.7 0.7 1.0"/>
+        </material>
+      </visual>
+      <collision>
+        <geometry>
+          <mesh filename="package://ur_description/meshes/ur3/collision/forearm.stl"/>
+        </geometry>
+      </collision>
+      <xacro:cylinder_inertial radius="0.075" length="${-a3}" mass="${forearm_mass}">
+        <origin xyz="0.0 0.0 ${-a3/2.0}" rpy="0 0 0" />
+      </xacro:cylinder_inertial>
+    </link>
+    <joint name="${prefix}wrist_1_joint" type="revolute">
+      <parent link="${prefix}forearm_link" />
+      <child link = "${prefix}wrist_1_link" />
+      <origin xyz="0.0 0.0 ${forearm_length}" rpy="0.0 ${pi / 2.0} 0.0" />
+      <axis xyz="0 1 0" />
+      <xacro:unless value="${joint_limited}">
+        <limit lower="${-2.0 * pi}" upper="${2.0 * pi}" effort="54.0" velocity="3.2"/>
+        <xacro:if value="${safety_limits}">
+          <safety_controller soft_lower_limit="${-2.0 * pi + safety_pos_margin}" soft_upper_limit="${2.0 * pi - safety_pos_margin}" k_position="${safety_k_position}" k_velocity="0.0"/>
+        </xacro:if>
+      </xacro:unless>
+      <xacro:if value="${joint_limited}">
+        <limit lower="${wrist_1_lower_limit}" upper="${wrist_1_upper_limit}" effort="54.0" velocity="3.2"/>
+        <xacro:if value="${safety_limits}">
+          <safety_controller soft_lower_limit="${wrist_1_lower_limit + safety_pos_margin}" soft_upper_limit="${wrist_1_upper_limit - safety_pos_margin}" k_position="${safety_k_position}" k_velocity="0.0"/>
+        </xacro:if>
+      </xacro:if>
+      <dynamics damping="0.0" friction="0.0"/>
+    </joint>
+    <link name="${prefix}wrist_1_link">
+      <visual>
+        <geometry>
+          <mesh filename="package://ur_description/meshes/ur3/visual/wrist1.dae"/>
+        </geometry>
+        <material name="LightGrey">
+          <color rgba="0.7 0.7 0.7 1.0"/>
+        </material>
+      </visual>
+      <collision>
+        <geometry>
+          <mesh filename="package://ur_description/meshes/ur3/collision/wrist1.stl"/>
+        </geometry>
+      </collision>
+      <xacro:cylinder_inertial radius="0.075" length="0.12" mass="${wrist_1_mass}">
+        <origin xyz="0.0 ${wrist_1_length} 0.0" rpy="0 0 0" />
+      </xacro:cylinder_inertial>
+    </link>
+    <joint name="${prefix}wrist_2_joint" type="revolute">
+      <parent link="${prefix}wrist_1_link" />
+      <child link = "${prefix}wrist_2_link" />
+      <origin xyz="0.0 ${wrist_1_length} 0.0" rpy="0.0 0.0 0.0" />
+      <axis xyz="0 0 1" />
+      <xacro:unless value="${joint_limited}">
+        <limit lower="${-2.0 * pi}" upper="${2.0 * pi}" effort="54.0" velocity="3.2"/>
+        <xacro:if value="${safety_limits}">
+          <safety_controller soft_lower_limit="${-2.0 * pi + safety_pos_margin}" soft_upper_limit="${2.0 * pi - safety_pos_margin}" k_position="${safety_k_position}" k_velocity="0.0"/>
+        </xacro:if>
+      </xacro:unless>
+      <xacro:if value="${joint_limited}">
+        <limit lower="${wrist_2_lower_limit}" upper="${wrist_2_upper_limit}" effort="54.0" velocity="3.2"/>
+        <xacro:if value="${safety_limits}">
+          <safety_controller soft_lower_limit="${wrist_2_lower_limit + safety_pos_margin}" soft_upper_limit="${wrist_2_upper_limit - safety_pos_margin}" k_position="${safety_k_position}" k_velocity="0.0"/>
+        </xacro:if>
+      </xacro:if>
+      <dynamics damping="0.0" friction="0.0"/>
+    </joint>
+    <link name="${prefix}wrist_2_link">
+      <visual>
+        <geometry>
+          <mesh filename="package://ur_description/meshes/ur3/visual/wrist2.dae"/>
+        </geometry>
+        <material name="LightGrey">
+          <color rgba="0.7 0.7 0.7 1.0"/>
+        </material>
+      </visual>
+      <collision>
+        <geometry>
+          <mesh filename="package://ur_description/meshes/ur3/collision/wrist2.stl"/>
+        </geometry>
+      </collision>
+      <xacro:cylinder_inertial radius="0.075" length="0.12" mass="${wrist_2_mass}">
+        <origin xyz="0.0 0.0 ${wrist_2_length}" rpy="0 0 0" />
+      </xacro:cylinder_inertial>
+    </link>
+    <joint name="${prefix}wrist_3_joint" type="revolute">
+      <parent link="${prefix}wrist_2_link" />
+      <child link = "${prefix}wrist_3_link" />
+      <origin xyz="0.0 0.0 ${wrist_2_length}" rpy="0.0 0.0 0.0" />
+      <axis xyz="0 1 0" />
+      <xacro:unless value="${joint_limited}">
+        <limit lower="${-2.0 * pi}" upper="${2.0 * pi}" effort="54.0" velocity="3.2"/>
+        <xacro:if value="${safety_limits}">
+          <safety_controller soft_lower_limit="${-2.0 * pi + safety_pos_margin}" soft_upper_limit="${2.0 * pi - safety_pos_margin}" k_position="${safety_k_position}" k_velocity="0.0"/>
+        </xacro:if>
+      </xacro:unless>
+      <xacro:if value="${joint_limited}">
+        <limit lower="${wrist_3_lower_limit}" upper="${wrist_3_upper_limit}" effort="54.0" velocity="3.2"/>
+        <xacro:if value="${safety_limits}">
+          <safety_controller soft_lower_limit="${wrist_3_lower_limit + safety_pos_margin}" soft_upper_limit="${wrist_3_upper_limit - safety_pos_margin}" k_position="${safety_k_position}" k_velocity="0.0"/>
+        </xacro:if>
+      </xacro:if>
+      <dynamics damping="0.0" friction="0.0"/>
+    </joint>
+    <link name="${prefix}wrist_3_link">
+      <visual>
+        <geometry>
+          <mesh filename="package://ur_description/meshes/ur3/visual/wrist3.dae"/>
+        </geometry>
+        <material name="LightGrey">
+          <color rgba="0.7 0.7 0.7 1.0"/>
+        </material>
+      </visual>
+      <collision>
+        <geometry>
+          <mesh filename="package://ur_description/meshes/ur3/collision/wrist3.stl"/>
+        </geometry>
+      </collision>
+      <xacro:cylinder_inertial radius="0.032" length="0.04" mass="${wrist_3_mass}">
+        <origin xyz="0.0 ${wrist_3_length - 0.02} 0.0" rpy="${pi/2} 0 0" />
+      </xacro:cylinder_inertial>
+    </link>
+    <joint name="${prefix}ee_fixed_joint" type="fixed">
+      <parent link="${prefix}wrist_3_link" />
+      <child link = "${prefix}ee_link" />
+      <origin xyz="0.0 ${wrist_3_length} 0.0" rpy="0.0 0.0 ${pi/2.0}" />
+    </joint>
+    <link name="${prefix}ee_link">
+      <collision>
+        <geometry>
+          <box size="0.01 0.01 0.01"/>
+        </geometry>
+        <origin rpy="0 0 0" xyz="-0.01 0 0"/>
+      </collision>
+    </link>
+    <xacro:ur_arm_transmission prefix="${prefix}" hw_interface="${transmission_hw_interface}" />
+    <xacro:ur_arm_gazebo prefix="${prefix}" />
+    <!-- ROS base_link to UR 'Base' Coordinates transform -->
+    <link name="${prefix}base"/>
+    <joint name="${prefix}base_link-base_fixed_joint" type="fixed">
+      <origin xyz="0 0 0" rpy="0 0 ${-pi}"/>
+      <parent link="${prefix}base_link"/>
+      <child link="${prefix}base"/>
+    </joint>
+    <!-- Frame coincident with all-zeros TCP on UR controller -->
+    <link name="${prefix}tool0"/>
+    <joint name="${prefix}wrist_3_link-tool0_fixed_joint" type="fixed">
+      <origin xyz="0 ${wrist_3_length} 0" rpy="${pi/-2.0} 0 0"/>
+      <parent link="${prefix}wrist_3_link"/>
+      <child link="${prefix}tool0"/>
+    </joint>
+        <!-- INSPECTION WINDOW-->
+    <link name="inspection_window">
+      <collision>
+        <geometry>
+          <mesh filename="file://$(find ur_description)/meshes/inspection_window.stl" scale="0.01 0.01 0.01"/>
+        </geometry>
+      </collision>
+      <visual>
+        <geometry>
+          <mesh filename="file://$(find ur_description)/meshes/inspection_window.stl" scale="0.01 0.01 0.01"/>
+        </geometry>
+      </visual>
+    </link>
+    <joint name="inspection_window_joint" type="fixed">
+      <parent link="right_panel_box"/>
+      <child link="inspection_window"/>
+      <origin xyz="-0.075 0.0 -0.15" rpy="1.5707 0.0 1.5707"/>
+    </joint>
+    <!-- INSPECTION WINDOW COVER-->
+    <link name="inspection_window_cover">
+      <collision>
+        <geometry>
+          <mesh filename="file://$(find ur_description)/meshes/inspection_window_cover.stl" scale="0.01 0.01 0.01"/>
+        </geometry>
+      </collision>
+      <visual>
+        <geometry>
+          <mesh filename="file://$(find ur_description)/meshes/inspection_window_cover.stl" scale="0.01 0.01 0.01"/>
+        </geometry>
+      </visual>
+    </link>
+    <joint name="inspection_window_cover_joint" type="fixed">
+      <parent link="inspection_window"/>
+      <child link="inspection_window_cover"/>
+      <origin xyz="0.0 0.059 0.0" rpy="0.0 0.0 0.0"/>
+    </joint>
     <!-- BOX macro -->
-    <xacro:macro name="boxes" params="prefix x y z width height depth color type">
+    <xacro:macro name="boxes" params="prefix x y z ox oy oz width height depth color type">
       <link name="${prefix}_box">
         <collision>
-          <origin xyz="${x} ${y} ${z}" rpy="0 0 0"/>
           <geometry>
             <box size="${width} ${height} ${depth}"/>
@@ -93,5 +403,4 @@
         </collision>
         <visual>
-          <origin xyz="${x} ${y} ${z}" rpy="0 0 0"/>
           <geometry>
             <box size="${width} ${height} ${depth}"/>
@@ -99,18 +408,9 @@
           <material name="${color}"/>
         </visual>
-        <inertial>
-          <origin xyz="0 0 0" rpy="0 0 0"/>
-          <mass value="1"/>
-          <inertia
-            ixx="0.004" ixy="0" ixz="0"
-            iyy="0.004" iyz="0"
-            izz="0.004"/>
-        </inertial>
       </link>
       <joint name="${prefix}_box_joint" type="${type}">
-        <origin xyz="0 0 0" rpy="0 0 0"/>
+        <origin xyz="${x} ${y} ${z}" rpy="${ox} ${oy} ${oz}"/>
         <parent link="world"/>
         <child link="${prefix}_box"/>
-        <limit effort="100" lower="-0.01" upper="0.06" velocity="0.05" />
       </joint>
       <gazebo reference="${prefix}_box">
@@ -120,270 +420,174 @@
     <!-- BOX macro -->
     <!-- BOX definition -->
-    <xacro:boxes prefix="0" x="0.0" y="0" z="-0.005" width="1.4" height="1.4" depth="0.01" color="White" type="fixed"/>
+    <xacro:boxes prefix="0" x="0.1" y="0" z="-0.105" ox="0" oy="0" oz="0" width="1.4" height="1.4" depth="0.01" color="LightGrey" type="fixed"/>
+    <xacro:boxes prefix="stand" x="0.0" y="0" z="-0.05" ox="0" oy="0" oz="0" width="0.15" height="0.15" depth="0.1" color="Grey" type="fixed"/>
+    <xacro:boxes prefix="center_panel" x="0.47" y="0" z="0.27" ox="0" oy="0" oz="0" width="0.02" height="0.3" depth="0.5" color="White" type="fixed"/>
+    <xacro:boxes prefix="left_panel" x="0.4265" y="0.2672" z="0.27" ox="0" oy="0" oz="0.3556" width="0.02" height="0.3" depth="0.5" color="White" type="fixed"/>
+    <xacro:boxes prefix="right_panel" x="0.4265" y="-0.2672" z="0.27" ox="0" oy="0" oz="-0.3556" width="0.02" height="0.3" depth="0.5" color="White" type="fixed"/>
+    <xacro:boxes prefix="IMU_module" x="0.21" y="0.2672" z="-0.075" ox="0" oy="0" oz="0.0" width="0.06" height="0.160" depth="0.05" color="Grey" type="fixed"/>
+<!--    <xacro:boxes prefix="Lid" x="0.3" y="-0.2672" z="0.05" ox="0" oy="0" oz="0.0" width="0.05" height="0.165" depth="0.005" color="Grey" type="fixed"/>-->
+<!--    <xacro:boxes prefix="Inspection_box" x="0.3" y="-0.2672" z="0.0" ox="0" oy="0" oz="0.0" width="0.05" height="0.165" depth="0.05" color="Grey" type="fixed"/>-->
     <!-- BOX definition -->
-    <joint name="${prefix}shoulder_pan_joint" type="revolute">
-      <parent link="${prefix}base_link" />
-      <child link = "${prefix}shoulder_link" />
-      <origin xyz="0.0 0.0 ${shoulder_height}" rpy="0.0 0.0 0.0" />
-      <axis xyz="0 0 1" />
-      <xacro:unless value="${joint_limited}">
-        <limit lower="${-2.0 * pi}" upper="${2.0 * pi}" effort="330.0" velocity="2.16"/>
-        <xacro:if value="${safety_limits}">
-          <safety_controller soft_lower_limit="${-2.0 * pi + safety_pos_margin}" soft_upper_limit="${2.0 * pi - safety_pos_margin}" k_position="${safety_k_position}" k_velocity="0.0"/>
-        </xacro:if>
-      </xacro:unless>
-      <xacro:if value="${joint_limited}">
-        <limit lower="${shoulder_pan_lower_limit}" upper="${shoulder_pan_upper_limit}" effort="330.0" velocity="2.16"/>
-        <xacro:if value="${safety_limits}">
-          <safety_controller soft_lower_limit="${shoulder_pan_lower_limit + safety_pos_margin}" soft_upper_limit="${shoulder_pan_upper_limit - safety_pos_margin}" k_position="${safety_k_position}" k_velocity="0.0"/>
-        </xacro:if>
-      </xacro:if>
-      <dynamics damping="0.0" friction="0.0"/>
-    </joint>
-    <link name="${prefix}shoulder_link">
-      <visual>
-        <geometry>
-          <mesh filename="package://ur_description/meshes/ur3/visual/shoulder.dae"/>
-        </geometry>
-        <material name="LightGrey">
-          <color rgba="0.7 0.7 0.7 1.0"/>
-        </material>
-      </visual>
-      <collision>
-        <geometry>
-          <mesh filename="package://ur_description/meshes/ur3/collision/shoulder.stl"/>
-        </geometry>
-      </collision>
-      <xacro:cylinder_inertial radius="0.075" length="0.178" mass="${shoulder_mass}">
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