Commit message: gripper2

File: ur_description/urdf/robotiq_arg2f.xacro (robot description, xacro)
@@ -1,6 +1,5 @@
 <?xml version="1.0"?>
 <robot xmlns:xacro="http://ros.org/wiki/xacro">
-  <!--xacro:include filename="$(find icl_phri_ur5_robotiq_arg140_description)/urdf/robotiq_arg2f_finger_tips.xacro" /-->
-  <xacro:macro name="robotiq_arg2f_base_link" params="prefix">
+  <xacro:macro name="base_link" params="prefix">
     <link name="${prefix}robotiq_arg2f_base_link">
       <inertial>

File: ur_description/urdf/robotiq_arg2f_140_model_macro.xacro (robot description, xacro)
@@ -47,16 +47,10 @@
       <visual>
         <origin xyz="0 0 0" rpy="0 0 0" />
-<!--        <geometry>-->
-<!--          <mesh filename="package://ur_description/meshes/gripper/robotiq_arg2f_${stroke}_outer_finger.stl" scale="1.0 0.6 0.6"/>-->
-<!--        </geometry>-->
-        <material name="">
-          <color rgba="0.1 0.1 0.1 1" />
-        </material>
-      </visual>
-      <collision>
-        <origin xyz="0 0 0" rpy="0 0 0" />
-<!--        <geometry>-->
-<!--          <mesh filename="package://ur_description/meshes/gripper/robotiq_arg2f_${stroke}_outer_finger.stl" scale="1.0 0.6 0.6"/>-->
-<!--        </geometry>-->
+        <material name="">
+          <color rgba="0.1 0.1 0.1 1" />
+        </material>
+      </visual>
+      <collision>
+        <origin xyz="0 0 0" rpy="0 0 0" />
       </collision>
     </link>
@@ -300,5 +294,5 @@
   <xacro:include filename="$(find ur_description)/urdf/robotiq_arg2f.xacro" />
   <xacro:macro name="robotiq_arg2f_140" params="prefix">
-    <xacro:robotiq_arg2f_base_link prefix="${prefix}"/>
+    <xacro:base_link prefix="${prefix}"/>
     <xacro:finger_links prefix="${prefix}" fingerprefix="left" stroke="140"/>
     <xacro:finger_links prefix="${prefix}" fingerprefix="right" stroke="140"/>

File: ur_description/urdf/ur3.urdf.xacro (robot description, xacro)
@@ -426,6 +426,4 @@
     <xacro:boxes prefix="right_panel" x="0.4265" y="-0.2672" z="0.27" ox="0" oy="0" oz="-0.3556" width="0.02" height="0.3" depth="0.5" color="White" type="fixed"/>
     <xacro:boxes prefix="IMU_module" x="0.21" y="0.2672" z="-0.075" ox="0" oy="0" oz="0.0" width="0.06" height="0.160" depth="0.05" color="Grey" type="fixed"/>
-<!--    <xacro:boxes prefix="Lid" x="0.3" y="-0.2672" z="0.05" ox="0" oy="0" oz="0.0" width="0.05" height="0.165" depth="0.005" color="Grey" type="fixed"/>-->
-<!--    <xacro:boxes prefix="Inspection_box" x="0.3" y="-0.2672" z="0.0" ox="0" oy="0" oz="0.0" width="0.05" height="0.165" depth="0.05" color="Grey" type="fixed"/>-->
     <!-- BOX definition -->
     <!-- CYLINDER macro -->
@@ -503,7 +501,4 @@
       <visual>
         <origin xyz="0 0 0" rpy="0 0 0" />
-<!--        <geometry>-->
-<!--          <mesh filename="package://ur_description/meshes/gripper/plate1.dae" scale="0.001 0.001 0.001"/>-->
-<!--        </geometry>-->
         <material name="">
           <color rgba="0.1 0.1 0.1 1" />
@@ -512,22 +507,11 @@
       <collision>
         <origin xyz="0 0 0" rpy="0 0 ${pi / 2}" />
-<!--        <geometry>-->
-<!--          <mesh filename="package://ur_description/meshes/gripper/plate1.dae" scale="0.01 0.01 0.01"/>-->
-<!--        </geometry>-->
       </collision>
     </link>
     <joint name="plate1_joint" type="fixed">
-<!--      <origin xyz="0.02 0.0 0.0304" rpy="3.141 1.5707 0.0" />-->
       <origin xyz="0.02 0.0 0.0304" rpy="3.141 1.5707 0.0" />
       <parent link="robotiq_arg2f_base_link" />
       <child link="plate1" />
      </joint>
-<!--    <xacro:include filename="$(find ur_description)/urdf/robotiq_arg2f_140_model_macro.xacro" />-->
-<!--    <xacro:robotiq_arg2f_140 prefix=""/>-->
-<!--    <joint name="${prefix}gripper" type="fixed">-->
-<!--      <origin xyz="0.0 0.0 0.0" rpy="0.0 0 0.0" />-->
-<!--      <parent link="plate1" />-->
-<!--      <child link="robotiq_arg2f_base_link" />-->
-<!--     </joint>-->
     <link name="camera_ur_mount">
       <visual>

Commit message: aruco

File: ur_description/urdf/robotiq_arg2f.xacro (robot description, xacro)
@@ -18,4 +18,7 @@
       </collision>
     </link>
+    <gazebo reference="${prefix}robotiq_arg2f_base_link">
+        <material>Gazebo/DarkGrey</material>
+    </gazebo>
   </xacro:macro>
   <xacro:macro name="finger_joints" params="prefix fingerprefix reflect">

File: ur_description/urdf/robotiq_arg2f_140_model_macro.xacro (robot description, xacro)
@@ -31,4 +31,7 @@
       </collision>
     </link>
+    <gazebo reference="${prefix}${fingerprefix}_outer_knuckle">
+        <material>Gazebo/DarkGrey</material>
+    </gazebo>
   </xacro:macro>
   <xacro:macro name="outer_finger" params="prefix fingerprefix stroke">
@@ -85,4 +88,7 @@
       </collision>
     </link>
+    <gazebo reference="${prefix}${fingerprefix}_inner_knuckle">
+        <material>Gazebo/DarkGrey</material>
+    </gazebo>
   </xacro:macro>
     <xacro:macro name="inner_knuckle2" params="prefix fingerprefix stroke">
@@ -115,4 +121,7 @@
       </collision>
     </link>
+    <gazebo reference="${prefix}${fingerprefix}_inner_knuckle2">
+        <material>Gazebo/DarkGrey</material>
+    </gazebo>
   </xacro:macro>
   <xacro:macro name="inner_finger" params="prefix fingerprefix stroke">
@@ -145,4 +154,7 @@
       </collision>
     </link>
+    <gazebo reference="${prefix}${fingerprefix}_inner_finger">
+        <material>Gazebo/DarkGrey</material>
+    </gazebo>
   </xacro:macro>
     <xacro:macro name="inner_finger2" params="prefix fingerprefix stroke">
@@ -175,4 +187,7 @@
       </collision>
     </link>
+    <gazebo reference="${prefix}${fingerprefix}_inner_finger2">
+        <material>Gazebo/DarkGrey</material>
+    </gazebo>
   </xacro:macro>
   <xacro:macro name="outer_finger_joint" params="prefix fingerprefix reflect">
@@ -272,4 +287,7 @@
       </collision>
     </link>
+    <gazebo reference="${prefix}${fingerprefix}_finger_tip">
+        <material>Gazebo/DarkGrey</material>
+    </gazebo>
   </xacro:macro>
   <link name="left_finger_tip_temp"/>

File: ur_description/urdf/ur3.urdf.xacro (robot description, xacro)
@@ -371,4 +371,7 @@
       </visual>
     </link>
+    <gazebo reference="inspection_window">
+        <material>Gazebo/Red</material>
+    </gazebo>
     <joint name="inspection_window_joint" type="fixed">
       <parent link="right_panel_box"/>
@@ -389,4 +392,7 @@
       </visual>
     </link>
+    <gazebo reference="inspection_window_cover">
+        <material>Gazebo/Red</material>
+    </gazebo>
     <joint name="inspection_window_cover_joint" type="fixed">
       <parent link="inspection_window"/>
@@ -408,4 +414,12 @@
           <material name="${color}"/>
         </visual>
+        <inertial>
+          <origin xyz="0 0 0" rpy="0 0 0"/>
+          <mass value="1"/>
+          <inertia
+            ixx="0.004" ixy="0" ixz="0"
+            iyy="0.004" iyz="0"
+            izz="0.004"/>
+        </inertial>
       </link>
       <joint name="${prefix}_box_joint" type="${type}">
@@ -441,4 +455,12 @@
           <material name="${color}"/>
         </visual>
+        <inertial>
+          <origin xyz="0 0 0" rpy="0 0 0"/>
+          <mass value="1"/>
+          <inertia
+            ixx="0.004" ixy="0" ixz="0"
+            iyy="0.004" iyz="0"
+            izz="0.004"/>
+        </inertial>
       </link>
       <joint name="${prefix}_cylinder_joint" type="${type}">
@@ -447,5 +469,5 @@
         <child link="${prefix}_cylinder"/>
       </joint>
-      <gazebo reference="${prefix}_box">
+      <gazebo reference="${prefix}_cylinder">
         <material>Gazebo/${color}</material>
       </gazebo>
@@ -470,4 +492,12 @@
         </geometry>
       </visual>
+      <inertial>
+        <origin xyz="0 0 0" rpy="0 0 0"/>
+        <mass value="1"/>
+        <inertia
+            ixx="0.004" ixy="0" ixz="0"
+            iyy="0.004" iyz="0"
+            izz="0.004"/>
+        </inertial>
     </link>
     <joint name="aruco_${prefix}_joint" type="fixed">
@@ -531,4 +561,7 @@
       </collision>
     </link>
+    <gazebo reference="camera_ur_mount">
+        <material>Gazebo/DarkGrey</material>
+    </gazebo>
     <joint name="camer_ur_mount_joint" type="fixed">
       <origin xyz="0.0 0.0 -0.0015" rpy="1.5707 0.0 -1.5707" />
@@ -569,4 +602,7 @@
       </collision>
     </link>
+    <gazebo reference="dys_middle">
+        <material>Gazebo/Grey</material>
+    </gazebo>
     <joint name="dys_middle_joint" type="fixed">
       <origin xyz="0.00375 0.0 0.02015" rpy="0.0 0.0 0.0" />
