Commit message: gripper_command

File: ur_description/urdf/robotiq_arg2f_140_model_macro.xacro (robot description, xacro)
@@ -242,5 +242,5 @@
       <child link="${prefix}left_outer_knuckle" />
       <axis xyz="-1 0 0" />
-      <limit lower="0" upper="1.31093125" velocity="2.0" effort="1000" />
+      <limit lower="0" upper="1.399" velocity="2.0" effort="1000" />
     </joint>
     <xacro:finger_joints prefix="${prefix}" fingerprefix="left" reflect="1.0"/>
